Commit message: Setup with pid controller

File: hyperdog_gazebo_sim/description/consts.xacro (robot description, xacro)
@@ -13,11 +13,11 @@
     <xacro:property name="use_dynamics" value="true"/>
     <xacro:macro name="hip_joint_dynamics">
-        <dynamics damping="0.01" friction="10000"/>
+        <dynamics damping="0.01" friction="0"/>
     </xacro:macro>
     <xacro:macro name="uleg_joint_dynamics">
-        <dynamics damping="0.01" friction="10000"/>
+        <dynamics damping="0.01" friction="0"/>
     </xacro:macro>
     <xacro:macro name="lleg_joint_dynamics">
-        <dynamics damping="0.01" friction="10000"/>
+        <dynamics damping="0.01" friction="0"/>
     </xacro:macro>
     <!-- configure inertia -->

File: hyperdog_gazebo_sim/description/gazebo_ros2_control_plugin.xacro (robot description, xacro)
@@ -14,11 +14,10 @@
 				name="gz_ros2_control::GazeboSimROS2ControlPlugin">
             <parameters>$(find hyperdog_gazebo_sim)/config/hyperdog_joint_controller.yaml</parameters>
-		    <robot_param>robot_description</robot_param>
-		    <robot_param_node>robot_state_publisher</robot_param_node>
-            <ros>
-		    	<argument>--ros-args</argument>
-		    	<argument>--params-file</argument>
-		    	<argument>$(find hyperdog_gazebo_sim)/config/ros2_control_gz_time.yaml</argument>
-		    </ros>
+			<robot_param_node>robot_state_publisher</robot_param_node>
+			<ros>
+				<argument>--ros-args</argument>
+				<argument>--params-file</argument>
+				<argument>$(find hyperdog_gazebo_sim)/config/ros2_control_gz_time.yaml</argument>
+			</ros>
         </plugin>
     </gazebo>
@@ -28,5 +27,5 @@
         </hardware>
         <joint name="FR_hip_joint">
-            <command_interface name="position">
+            <command_interface name="effort">
                 <param name="min">-1.57</param>
                 <param name="max">1.57</param>
@@ -39,5 +38,5 @@
         </joint>
         <joint name="FR_uleg_joint">
-            <command_interface name="position">
+            <command_interface name="effort">
                 <param name="min">-1.2217</param>
                 <param name="max">3.14</param>
@@ -50,5 +49,5 @@
         </joint>
         <joint name="FR_lleg_joint">
-            <command_interface name="position">
+            <command_interface name="effort">
                 <param name="min">0.45</param>
                 <param name="max">2.3562</param>
@@ -61,5 +60,5 @@
         </joint>
         <joint name="FL_hip_joint">
-            <command_interface name="position">
+            <command_interface name="effort">
                 <param name="min">-1.57</param>
                 <param name="max">1.57</param>
@@ -72,5 +71,5 @@
         </joint>
         <joint name="FL_uleg_joint">
-            <command_interface name="position">
+            <command_interface name="effort">
                 <param name="min">-1.2217</param>
                 <param name="max">3.14</param>
@@ -83,5 +82,5 @@
         </joint>
         <joint name="FL_lleg_joint">
-            <command_interface name="position">
+            <command_interface name="effort">
                 <param name="min">0.45</param>
                 <param name="max">2.3562</param>
@@ -94,5 +93,5 @@
         </joint>
         <joint name="BR_hip_joint">
-            <command_interface name="position">
+            <command_interface name="effort">
                 <param name="min">-1.57</param>
                 <param name="max">1.57</param>
@@ -105,5 +104,5 @@
         </joint>
         <joint name="BR_uleg_joint">
-            <command_interface name="position">
+            <command_interface name="effort">
                 <param name="min">-1.2217</param>
                 <param name="max">3.14</param>
@@ -116,5 +115,5 @@
         </joint>
         <joint name="BR_lleg_joint">
-            <command_interface name="position">
+            <command_interface name="effort">
                 <param name="min">0.45</param>
                 <param name="max">2.3562</param>
@@ -127,5 +126,5 @@
         </joint>
         <joint name="BL_hip_joint">
-            <command_interface name="position">
+            <command_interface name="effort">
                 <param name="min">-1.57</param>
                 <param name="max">1.57</param>
@@ -138,5 +137,5 @@
         </joint>
         <joint name="BL_uleg_joint">
-            <command_interface name="position">
+            <command_interface name="effort">
                 <param name="min">-1.2217</param>
                 <param name="max">3.14</param>
@@ -149,5 +148,5 @@
         </joint>
         <joint name="BL_lleg_joint">
-            <command_interface name="position">
+            <command_interface name="effort">
                 <param name="min">0.45</param>
                 <param name="max">2.3562</param>
